Commit message: Fix joint name | Add comments to source of mass and inertia

File: end_effectors/ft_sensors/ati_mini45.urdf.xacro (robot description, xacro)
@@ -9,5 +9,5 @@
     <xacro:property name="length" value="0.0327" />
     <xacro:property name="ee_inertials" value="${sensor_inertials}" />
-    <joint name="${prefix}hand_joint" type="fixed">
+    <joint name="${prefix}ati_mini45_base_joint" type="fixed">
       <parent link="${parent_link}" />
       <child link="${prefix}ati_mini45" />

Commit message: Move ft sensor as part of franka robot | Add basic Gazebo support

File: end_effectors/ft_sensors/ati_mini45.urdf.xacro (robot description, xacro)
@@ -3,6 +3,7 @@
   <xacro:include filename="$(find franka_description)/end_effectors/common/utils.xacro" />
   <xacro:include filename="$(find franka_description)/end_effectors/common/ee_with_one_link.xacro" />
+  <xacro:include filename="$(find franka_description)/end_effectors/ft_sensors/ati_mini45_arguments.xacro"/>
   <xacro:macro name="ati_mini45"
-    params="prefix parent_link rpy_sensor:='0 0 0' xyz_sensor:='0 0 0' ip_address rdt_sampling_rate internal_filter_rate use_hardware_biasing sensor_inertials safety_distance:=0 gazebo:=false description_pkg:=franka_description with_sc:=false">
+    params="prefix parent_link rpy_sensor:='0 0 0' xyz_sensor:='0 0 0' ip_address rdt_sampling_rate internal_filter_rate use_hardware_biasing sensor_inertials safety_distance:=0 gazebo:=false description_pkg:=franka_description with_sc:=false measurement_frame_name:='ati_mini45_measurement_reference'">
     <!-- length and radius of the sensor with mounting plates -->
     <xacro:property name="radius" value="0.0315" />
@@ -51,18 +52,19 @@
     </joint>
     <link name="${prefix}ati_mini45_tool_mount" />
-    <joint name="${prefix}ati_mini45_measurement_reference_joint" type="fixed">
+    <joint name="${measurement_frame_name}_joint" type="fixed">
       <parent link="${prefix}ati_mini45" />
-      <child link="${prefix}ati_mini45_measurement_reference" />
-      <origin xyz="0 0 ${length / 2}" rpy="0 0 0" />
+      <child link="${measurement_frame_name}" />
+      <origin xyz="0 0 ${length / 2}" rpy="${pi} 0.0 ${pi / 3 * 2}" />
     </joint>
-    <link name="${prefix}ati_mini45_measurement_reference" />
-    <xacro:include filename="$(find net_ft_description)/urdf/net_ft_sensor.ros2_control.xacro" />
-    <xacro:net_ft_sensor_ros2_control
-      name="NetFtHardwareInterface"
-      sensor_type="ati"
-      ip_address="${ip_address}"
-      rdt_sampling_rate="${rdt_sampling_rate}"
-      internal_filter_rate="${internal_filter_rate}"
-      use_hardware_biasing="${use_hardware_biasing}" />
+    <link name="${measurement_frame_name}" />
+    <xacro:unless value="${gazebo}">
+      <xacro:include filename="$(find franka_description)/end_effectors/ft_sensors/ati_mini45.ros2_control.urdf.xacro"/>
+      <xacro:net_ft_sensor_ros2_control
+          ip_address="${ip_address}"
+          rdt_sampling_rate="${rdt_sampling_rate}"
+          internal_filter_rate="${internal_filter_rate}"
+          use_hardware_biasing="${use_hardware_biasing}"
+          ft_sensor_frame_name="${measurement_frame_name}"/>
+    </xacro:unless>
   </xacro:macro>
 </robot>

File: robots/common/franka_arm.ros2_control.xacro (robot description, xacro)
@@ -11,5 +11,7 @@
              gazebo_effort:=^|false
              arm_prefix:=''
-             multi_arm:=false">
+             multi_arm:=false
+             use_ft_sensor:=^|false
+             ft_sensor_frame_name:=''">
     <xacro:property name="arm_prefix_modified" value="${'' if arm_prefix == '' else arm_prefix + '_'}" />
     <ros2_control name="${arm_prefix_modified}FrankaHardwareInterface" type="system">
@@ -64,4 +66,13 @@
         </joint>
       </xacro:macro>
+      <!-- Gauss noise macro -->
+      <xacro:macro name="gauss_noise" params="stddev:=0.0">
+        <noise type="gaussian">
+          <mean>0.0</mean>
+          <stddev>${stddev}</stddev>
+          <bias_mean>0.0</bias_mean>
+          <bias_stddev>0.0</bias_stddev>
+        </noise>
+      </xacro:macro>
       <xacro:configure_joint joint_name="${arm_prefix_modified}${arm_id}_joint1" initial_position="0.0"/>
       <xacro:configure_joint joint_name="${arm_prefix_modified}${arm_id}_joint2" initial_position="${-pi/4}"/>
@@ -74,4 +85,15 @@
         <xacro:configure_joint joint_name="${arm_id}_finger_joint1" initial_position="0.0" />
         <xacro:configure_joint joint_name="${arm_id}_finger_joint2" mimic_joint="${arm_id}_finger_joint1"/>
+      </xacro:if>
+      <xacro:if value="${gazebo and use_ft_sensor}">
+        <sensor name="ati_mini45">
+          <state_interface name="force.x"/>
+          <state_interface name="force.y"/>
+          <state_interface name="force.z"/>
+          <state_interface name="torque.x"/>
+          <state_interface name="torque.y"/>
+          <state_interface name="torque.z"/>
+          <param name="frame_id">${ft_sensor_frame_name}</param>
+        </sensor>
       </xacro:if>
     </ros2_control>
@@ -97,4 +119,35 @@
         </plugin>
       </gazebo>
+      <!-- For now ft-sensor in gazebo doesn't seem to work. Even though the syntax for the sensor seems to match-->
+      <!-- what can be found in unit tests of the Gazebo and sensor is registered in the UI of Gazebo. -->
+      <gazebo reference="${arm_prefix_modified}${arm_id}_joint7">
+        <sensor name="ati_mini45" type="force_torque">
+          <alwaysOn>1</alwaysOn>
+          <update_rate>1000</update_rate>
+          <visualize>1</visualize>
+          <frame>${ft_sensor_frame_name}</frame>
+          <ignition_frame_id>${ft_sensor_frame_name}</ignition_frame_id>
+          <topic>force_torque</topic>
+          <force_torque>
+            <frame>child</frame>
+            <measure_direction>child_to_parent</measure_direction>
+            <!-- <measure_direction>parent_to_child</measure_direction> -->
+            <!-- check the sign of the force along -Y or +Y -->
+            <force>
+              <!-- N -->
+              <x><xacro:gauss_noise stddev="0.23810"/></x>
+              <y><xacro:gauss_noise stddev="0.20312"/></y>
+              <z><xacro:gauss_noise stddev="0.40506"/></z>
+            </force>
+            <torque>
+              <!-- Nm -->
+              <x><xacro:gauss_noise stddev="0.00167"/></x>
+              <y><xacro:gauss_noise stddev="0.00096"/></y>
+              <z><xacro:gauss_noise stddev="0.00267"/></z>
+            </torque>
+          </force_torque>
+          <!-- Values measured on the real sensor -->
+        </sensor>
+      </gazebo>
     </xacro:if>
   </xacro:macro>

File: robots/common/franka_robot.xacro (robot description, xacro)
@@ -23,6 +23,6 @@
                       arm_prefix:=''
                       connected_to:='base'
-                      multi_arm:=false"
-                      >
+                      multi_arm:=false
+                      use_ft_sensor:='false'">
     <xacro:include filename="$(find franka_description)/robots/common/utils.xacro" />
     <xacro:include filename="$(find franka_description)/robots/common/franka_arm.xacro" />
@@ -43,4 +43,23 @@
       connected_to="${connected_to}"
     />
+    <xacro:if value="${use_ft_sensor}">
+      <xacro:include filename="$(find franka_description)/end_effectors/ft_sensors/ati_mini45.urdf.xacro" />
+      <xacro:include filename="$(find franka_description)/end_effectors/ft_sensors/ati_mini45_arguments.xacro" />
+      <xacro:property name="ft_sensor_measurement_frame_name" value="${arm_prefix_modified}ati_mini45_measurement_reference" />
+      <xacro:ati_mini45
+        parent_link="fer_link8"
+        prefix="${arm_prefix_modified}"
+        ip_address="$(arg ft_sensor_ip)"
+        gazebo="${gazebo}"
+        rdt_sampling_rate="$(arg rdt_sampling_rate)"
+        internal_filter_rate="$(arg internal_filter_rate)"
+        use_hardware_biasing="$(arg use_hardware_biasing)"
+        sensor_inertials="${xacro.load_yaml('$(find franka_description)/end_effectors/ft_sensors/inertials.yaml')}"
+        measurement_frame_name="${ft_sensor_measurement_frame_name}">
+      </xacro:ati_mini45>
+    </xacro:if>
+    <xacro:unless value="${use_ft_sensor}">
+      <xacro:property name="ft_sensor_measurement_frame_name" value="${arm_prefix_modified}ati_mini45_measurement_reference" />
+    </xacro:unless>
     <xacro:if value="${hand and ee_id == 'franka_hand'}">
       <xacro:include filename="$(find franka_description)/end_effectors/common/franka_hand.xacro"/>
@@ -54,5 +73,6 @@
       </xacro:if>
       <xacro:property name="special_connection" value="$(arg special_connection)" />
-      <xacro:property name="connection" value="${special_connection if special_connection != '' else arm_id + '_link8'}" />
+      <xacro:property name="default_connection" value="${(arm_id + '_link8') if not use_ft_sensor else 'ati_mini45_tool_mount'}" />
+      <xacro:property name="connection" value="${special_connection if special_connection != '' else default_connection}" />
       <xacro:franka_hand
         connected_to="${arm_prefix_modified}${connection}"
@@ -75,6 +95,6 @@
       <xacro:include filename="$(find franka_description)/end_effectors/common/utils.xacro" />
       <xacro:include filename="$(find franka_description)/end_effectors/$(arg ee_id)/$(arg ee_id)_arguments.xacro" />
-      <xacro:property name="special_connection" value="$(arg special_connection)" />
-      <xacro:property name="connection" value="${special_connection if special_connection == '' else arm_id + '_link8'}" />
+      <xacro:property name="default_connection" value="${(arm_id + '_link8') if not use_ft_sensor else 'ati_mini45_tool_mount'}" />
+      <xacro:property name="connection" value="${special_connection if special_connection != '' else default_connection}" />
       <xacro:ee_with_one_link
         connected_to="${arm_prefix_modified}${connection}"
@@ -203,4 +223,6 @@
           arm_prefix="${arm_prefix}"
           multi_arm="$(arg multi_arm)"
+          use_ft_sensor="${use_ft_sensor}"
+          ft_sensor_frame_name="${ft_sensor_measurement_frame_name}"
       />
     </xacro:if>

File: robots/fer/fer.urdf.xacro (robot description, xacro)
@@ -2,5 +2,4 @@
 <robot xmlns:xacro="http://www.ros.org/wiki/xacro" name="fer">
   <xacro:include filename="$(find franka_description)/robots/common/franka_robot.xacro"/>
-  <xacro:include filename="$(find franka_description)/end_effectors/ft_sensors/ati_mini45.urdf.xacro" />
   <!--
     DEPRECATION NOTICE
@@ -36,10 +35,10 @@
   <!-- Should fake sensors be used? -->
   <xacro:arg name="fake_sensor_commands" default="false" />
-  <!-- Should the robot be spawned in Gazebo with effort interfaces?" -->
+  <!-- Should the robot be spawned in Gazebo with effort interfaces? -->
   <xacro:arg name="gazebo_effort" default="false" />
   <!-- For a multi arm setup, we need a threaded robot running async-->
   <xacro:arg name="multi_arm" default="false" />
-  <!-- IP address or hostname of the force-torque sensor" -->
-  <xacro:arg name="ft_sensor_ip" default="" />
+  <!-- Should force torque sensors be used? -->
+  <xacro:arg name="use_ft_sensor" default="false" />
   <xacro:franka_robot arm_id="fer"
                       joint_limits="${xacro.load_yaml('$(find franka_description)/robots/fer/joint_limits.yaml')}"
@@ -58,18 +57,7 @@
                       gazebo_effort="$(arg gazebo_effort)"
                       no_prefix="$(arg no_prefix)"
-                      arm_prefix= ""
-                      connected_to= "base">
+                      arm_prefix=""
+                      connected_to="base"
+                      use_ft_sensor="$(arg use_ft_sensor)">
   </xacro:franka_robot>
-  <!-- ATI sensors have sampling rate as 7000 divided by an integer -->
-  <!-- Dividing by 3 is the closest to 2 times 1000 Hz which is the -->
-  <!-- control frequency of Panda -->
-  <xacro:property name="rdt_sampling_rate" value="${int(7000 / 3)}" />
-  <xacro:ati_mini45 parent_link="fer_link8"
-                    prefix=""
-                    ip_address="$(arg ft_sensor_ip)"
-                    rdt_sampling_rate="${rdt_sampling_rate}"
-                    internal_filter_rate="0"
-                    use_hardware_biasing="false"
-                    sensor_inertials="${xacro.load_yaml('$(find franka_description)/end_effectors/ft_sensors/inertials.yaml')}">
-  </xacro:ati_mini45>
 </robot>

Commit message: Fix force sensor measurements

File: end_effectors/ft_sensors/ati_mini45.urdf.xacro (robot description, xacro)
@@ -46,10 +46,4 @@
       </joint>
     </xacro:if>
-    <joint name="${prefix}ati_mini45_tool_mount_joint" type="fixed">
-      <parent link="${prefix}ati_mini45" />
-      <child link="${prefix}ati_mini45_tool_mount" />
-      <origin xyz="0 0 ${length}" rpy="0 0 0" />
-    </joint>
-    <link name="${prefix}ati_mini45_tool_mount" />
     <joint name="${measurement_frame_name}_joint" type="fixed">
       <parent link="${prefix}ati_mini45" />
@@ -58,4 +52,10 @@
     </joint>
     <link name="${measurement_frame_name}" />
+    <joint name="${prefix}ati_mini45_tool_mount_joint" type="fixed">
+      <parent link="${measurement_frame_name}" />
+      <child link="${prefix}ati_mini45_tool_mount" />
+      <origin xyz="0 0 ${-length / 2}" rpy="${pi} 0.0 ${pi / 3 * 2}" />
+    </joint>
+    <link name="${prefix}ati_mini45_tool_mount" />
     <xacro:unless value="${gazebo}">
       <xacro:include filename="$(find franka_description)/end_effectors/ft_sensors/ati_mini45.ros2_control.urdf.xacro"/>

File: robots/common/franka_arm.ros2_control.xacro (robot description, xacro)
@@ -122,6 +122,5 @@
       <!-- For now ft-sensor in gazebo doesn't seem to work. Even though the syntax for the sensor seems to match-->
       <!-- what can be found in unit tests of the Gazebo and sensor is registered in the UI of Gazebo. -->
-      <!-- <gazebo reference="${ft_sensor_frame_name}_joint"> -->
-       <gazebo reference="${arm_prefix_modified}${arm_id}_joint7">
+      <gazebo reference="${ft_sensor_frame_name}_joint">
         <provideFeedback>true</provideFeedback>
         <preserveFixedJoint>true</preserveFixedJoint>
@@ -134,8 +133,7 @@
           <topic>force_torque</topic>
           <force_torque>
-            <frame>child</frame>
+            <frame>parent</frame>
             <measure_direction>child_to_parent</measure_direction>
-            <!-- <measure_direction>parent_to_child</measure_direction> -->
-            <!-- check the sign of the force along -Y or +Y -->
+            <!-- Values measured on the real sensor -->
             <force>
               <!-- N -->
@@ -151,5 +149,4 @@
             </torque>
           </force_torque>
-          <!-- Values measured on the real sensor -->
         </sensor>
       </gazebo>
