Commit message: Add mass to end effector tip

File: end_effectors/ati_mini45_with_camera/ati_mini45_with_camera.urdf.xacro (robot description, xacro)
@@ -58,5 +58,7 @@
       <origin xyz="0 0 0.073915" rpy="${pi} 0.0 ${pi / 3 * 2}" />
     </joint>
-    <link name="${prefix_expanded}ati_mini45_with_camera_tool_mount" />
+    <link name="${prefix_expanded}ati_mini45_with_camera_tool_mount">
+      <xacro:ee-inertials name="ati_mini45_with_camera_tip" />
+    </link>
     <xacro:unless value="${gazebo}">
       <xacro:include filename="$(find franka_description)/end_effectors/ft_sensors/ati_mini45.ros2_control.urdf.xacro"/>

File: robots/common/franka_robot.xacro (robot description, xacro)
@@ -98,5 +98,4 @@
       <xacro:property name="special_connection" value="$(arg special_connection)" />
       <xacro:property name="default_connection" value="${arm_id + '_link8'}" />
-      <xacro:property name="connection" value="${special_connection if special_connection != '' else default_connection}" />
       <xacro:ati_mini45_with_camera
           parent_link="${arm_prefix_modified}${default_connection}"

Commit message: Rename tool_mount and tip to tool frame

File: end_effectors/ati_mini45_with_camera/ati_mini45_with_camera.urdf.xacro (robot description, xacro)
@@ -53,11 +53,11 @@
     </joint>
     <link name="${measurement_frame_name}" />
-    <joint name="${prefix_expanded}ati_mini45_with_camera_tool_mount_joint" type="fixed">
+    <joint name="${prefix_expanded}ati_mini45_with_camera_tool_joint" type="fixed">
       <parent link="${measurement_frame_name}" />
-      <child link="${prefix_expanded}ati_mini45_with_camera_tool_mount" />
+      <child link="${prefix_expanded}ati_mini45_with_camera_tool" />
       <origin xyz="0 0 0.073915" rpy="${pi} 0.0 ${pi / 3 * 2}" />
     </joint>
-    <link name="${prefix_expanded}ati_mini45_with_camera_tool_mount">
-      <xacro:ee-inertials name="ati_mini45_with_camera_tip" />
+    <link name="${prefix_expanded}ati_mini45_with_camera_tool">
+      <xacro:ee-inertials name="ati_mini45_with_camera_tool" />
     </link>
     <xacro:unless value="${gazebo}">

Commit message: Fix tool placement in Z

File: end_effectors/ati_mini45_with_camera/ati_mini45_with_camera.urdf.xacro (robot description, xacro)
@@ -56,5 +56,5 @@
       <parent link="${measurement_frame_name}" />
       <child link="${prefix_expanded}ati_mini45_with_camera_tool" />
-      <origin xyz="0 0 0.073915" rpy="${pi} 0.0 ${pi / 3 * 2}" />
+      <origin xyz="0 0 -0.073915" rpy="${pi} 0.0 ${pi / 3 * 2}" />
     </joint>
     <link name="${prefix_expanded}ati_mini45_with_camera_tool">

Commit message: Fix ft sensor + hand configuration | Fix sensor rotation

File: end_effectors/ati_mini45_with_camera/ati_mini45_with_camera.urdf.xacro (robot description, xacro)
@@ -50,5 +50,5 @@
       <parent link="${prefix_expanded}ati_mini45_with_camera" />
       <child link="${measurement_frame_name}" />
-      <origin xyz="0 0 0.017785" rpy="${pi} 0.0 ${pi / 3 * 2}" />
+      <origin xyz="0 0 0.017785" rpy="${pi} 0.0 ${(pi / 4) + (pi / 3 * 2)}" />
     </joint>
     <link name="${measurement_frame_name}" />

File: robots/common/franka_robot.xacro (robot description, xacro)
@@ -49,5 +49,5 @@
         <xacro:include filename="$(find franka_description)/end_effectors/ft_sensors/ati_mini45_arguments.xacro" />
         <xacro:ati_mini45
-          parent_link="${arm_prefix_modified}_link8"
+          parent_link="${arm_id}_link8"
           prefix="${arm_prefix_modified}"
           ip_address="$(arg ft_sensor_ip)"
@@ -96,5 +96,4 @@
       <xacro:include filename="$(find franka_description)/end_effectors/$(arg ee_id)/$(arg ee_id).urdf.xacro" />
       <xacro:include filename="$(find franka_description)/end_effectors/$(arg ee_id)/$(arg ee_id)_arguments.xacro" />
-      <xacro:property name="special_connection" value="$(arg special_connection)" />
       <xacro:property name="default_connection" value="${arm_id + '_link8'}" />
       <xacro:ati_mini45_with_camera
@@ -151,5 +150,5 @@
     <!-- use_mesh="true" produces an error when visualizing with rviz2
     because the generated urdf contains mesh filename paths that do not start with file:// -->
-    <xacro:sensor_d435 parent="${arm_id}_ref_camera_link" name="camera" use_nominal_extrinsics="true" use_mesh="true">
+    <xacro:sensor_d435 parent="${arm_id}_ref_camera_link" name="camera" use_nominal_extrinsics="true" use_mesh="false">
       <origin xyz="0 0 0" rpy="0 0 0"/>
     </xacro:sensor_d435>

Commit message: Add end effector tip collision as a sphere

File: end_effectors/ati_mini45_with_camera/ati_mini45_with_camera.urdf.xacro (robot description, xacro)
@@ -28,5 +28,4 @@
             filename="package://${description_pkg}/meshes/robot_ee/ati_mini45_with_camera/visual/ati_mini45_with_camera.stl" />
         </geometry>
-        <origin xyz="0 0 ${length / 2}" rpy="0 0 0" />
       </collision>
       <xacro:ee-inertials name="ati_mini45_with_camera_base" />
@@ -59,4 +58,9 @@
     </joint>
     <link name="${prefix_expanded}ati_mini45_with_camera_tool">
+      <collision name="${prefix_expanded}ati_mini45_with_camera_collision">
+        <geometry>
+          <sphere radius="0.013"/>
+        </geometry>
+      </collision>
       <xacro:ee-inertials name="ati_mini45_with_camera_tool" />
     </link>
