Commit message: add camera mound stl, realsense and default camera extrinsics parameters

File: robots/common/franka_robot.xacro (robot description, xacro)
@@ -23,5 +23,6 @@
                       arm_prefix:=''
                       connected_to:='base'
-                      multi_arm:=false">
+                      multi_arm:=false"
+                      >
     <xacro:include filename="$(find franka_description)/robots/common/utils.xacro" />
     <xacro:include filename="$(find franka_description)/robots/common/franka_arm.xacro" />
@@ -92,4 +93,49 @@
       />
     </xacro:if>
+    <!-- D435 camera -->
+    <!-- TODO: pass location of calibrated-params -->
+    <xacro:property name="camera_pose_file"
+                    value="$(find franka_description)/robots/${arm_id}/calibrated-params.yaml" />
+    <xacro:property name="camera_pose" value="${xacro.load_yaml(camera_pose_file)}"/>
+    <link name="${arm_id}_ref_camera_link"/>
+    <joint name="${arm_id}_ref_camera_joint" type="fixed">
+      <parent link="${arm_id}_hand"/>
+      <child link="${arm_id}_ref_camera_link"/>
+      <origin xyz="${camera_pose['camera']['x']}
+                    ${camera_pose['camera']['y']}
+                    ${camera_pose['camera']['z']}"
+        rpy="${camera_pose['camera']['roll']}
+                    ${camera_pose['camera']['pitch']}
+                    ${camera_pose['camera']['yaw']}"/>
+    </joint>
+    <xacro:include filename="$(find realsense2_description)/urdf/_d435.urdf.xacro" />
+    <xacro:sensor_d435 parent="${arm_id}_ref_camera_link" name="camera" use_nominal_extrinsics="true">
+      <origin xyz="0 0 0" rpy="0 0 0"/>
+    </xacro:sensor_d435>
+    <!-- camera support -->
+    <link name="${arm_id}_camera_support_link">
+      <inertial>
+        <mass value="0.010"/>
+        <origin xyz="0 0 0"/>
+        <inertia ixx="0.001" iyy="0.001" izz="0.001" ixy="0" iyz="0" ixz="0"/>
+      </inertial>
+      <visual>
+        <origin xyz="0.022 0 -0.012" rpy="3.141592653589793 0 -1.5707963267948966"/>
+        <geometry>
+          <mesh filename="$(find franka_description)/meshes/camera-support.stl" scale="1 1 1"/>
+        </geometry>
+      </visual>
+      <collision>
+        <origin xyz="0.022 0 -0.012" rpy="3.141592653589793 0 -1.5707963267948966"/>
+        <geometry>
+          <mesh filename="$(find franka_description)/meshes/camera-support.stl" scale="1 1 1"/>
+        </geometry>
+      </collision>
+    </link>
+    <joint name="${arm_id}_camera_support_joint" type="fixed">
+      <parent link="${arm_id}_hand"/>
+      <child link="${arm_id}_camera_support_link"/>
+      <origin xyz="0 0 0" rpy="3.141592653589793 0 0"/>
+    </joint>
     <!-- Definition of additional Gazebo tags -->
     <xacro:if value="${gazebo}">

Commit message: fix rviz camera mount stl issue + make it black

File: robots/common/franka_robot.xacro (robot description, xacro)
@@ -123,11 +123,14 @@
         <origin xyz="0.022 0 -0.012" rpy="3.141592653589793 0 -1.5707963267948966"/>
         <geometry>
-          <mesh filename="$(find franka_description)/meshes/camera-support.stl" scale="1 1 1"/>
+          <mesh filename="file://$(find franka_description)/meshes/camera-support.stl" scale="1 1 1"/>
         </geometry>
+        <material name="camera_support">
+          <color rgba="0 0.0 0.0 1.0"/>
+        </material>
       </visual>
       <collision>
         <origin xyz="0.022 0 -0.012" rpy="3.141592653589793 0 -1.5707963267948966"/>
         <geometry>
-          <mesh filename="$(find franka_description)/meshes/camera-support.stl" scale="1 1 1"/>
+          <mesh filename="file://$(find franka_description)/meshes/camera-support.stl" scale="1 1 1"/>
         </geometry>
       </collision>

Commit message: use package:// prefix instead of file://

File: robots/common/franka_robot.xacro (robot description, xacro)
@@ -125,5 +125,5 @@
         <origin xyz="0.022 0 -0.012" rpy="3.141592653589793 0 -1.5707963267948966"/>
         <geometry>
-          <mesh filename="file://$(find franka_description)/meshes/camera-support.stl" scale="1 1 1"/>
+          <mesh filename="package://franka_description/meshes/camera-support.stl" />
         </geometry>
         <material name="camera_support">
@@ -134,5 +134,5 @@
         <origin xyz="0.022 0 -0.012" rpy="3.141592653589793 0 -1.5707963267948966"/>
         <geometry>
-          <mesh filename="file://$(find franka_description)/meshes/camera-support.stl" scale="1 1 1"/>
+          <mesh filename="package://franka_description/meshes/camera-support.stl" />
         </geometry>
       </collision>

Commit message: Add deburring end effector with LAAS camera calibration

File: robots/common/franka_robot.xacro (robot description, xacro)
@@ -44,18 +44,19 @@
     />
     <xacro:if value="${use_ft_sensor}">
-      <xacro:include filename="$(find franka_description)/end_effectors/ft_sensors/ati_mini45.urdf.xacro" />
-      <xacro:include filename="$(find franka_description)/end_effectors/ft_sensors/ati_mini45_arguments.xacro" />
       <xacro:property name="ft_sensor_measurement_frame_name" value="${arm_prefix_modified}ati_mini45_measurement_reference" />
-      <xacro:ati_mini45
-        parent_link="fer_link8"
-        prefix="${arm_prefix_modified}"
-        ip_address="$(arg ft_sensor_ip)"
-        gazebo="${gazebo}"
-        rdt_sampling_rate="$(arg rdt_sampling_rate)"
-        internal_filter_rate="$(arg internal_filter_rate)"
-        use_hardware_biasing="$(arg use_hardware_biasing)"
-        sensor_inertials="${xacro.load_yaml('$(find franka_description)/end_effectors/ft_sensors/inertials.yaml')}"
-        measurement_frame_name="${ft_sensor_measurement_frame_name}">
-      </xacro:ati_mini45>
+      <xacro:if value="${hand and ee_id != 'ati_mini45_with_camera'}">
+        <xacro:include filename="$(find franka_description)/end_effectors/ft_sensors/ati_mini45.urdf.xacro" />
+        <xacro:include filename="$(find franka_description)/end_effectors/ft_sensors/ati_mini45_arguments.xacro" />
+        <xacro:ati_mini45
+          parent_link="${arm_prefix_modified}_link8"
+          prefix="${arm_prefix_modified}"
+          ip_address="$(arg ft_sensor_ip)"
+          gazebo="${gazebo}"
+          rdt_sampling_rate="$(arg rdt_sampling_rate)"
+          internal_filter_rate="$(arg internal_filter_rate)"
+          use_hardware_biasing="$(arg use_hardware_biasing)"
+          sensor_inertials="${xacro.load_yaml('$(find franka_description)/end_effectors/ft_sensors/inertials.yaml')}"
+          measurement_frame_name="${ft_sensor_measurement_frame_name}" />
+      </xacro:if>
     </xacro:if>
     <xacro:unless value="${use_ft_sensor}">
@@ -91,12 +92,31 @@
       />
     </xacro:if>
-    <xacro:if value="${hand and ee_id != 'none' and ee_id != 'franka_hand'}">
+    <xacro:if value="${hand and ee_id == 'ati_mini45_with_camera'}">
+      <xacro:include filename="$(find franka_description)/end_effectors/common/utils.xacro" />
+      <xacro:include filename="$(find franka_description)/end_effectors/$(arg ee_id)/$(arg ee_id).urdf.xacro" />
+      <xacro:include filename="$(find franka_description)/end_effectors/$(arg ee_id)/$(arg ee_id)_arguments.xacro" />
+      <xacro:property name="special_connection" value="$(arg special_connection)" />
+      <xacro:property name="default_connection" value="${arm_id + '_link8'}" />
+      <xacro:property name="connection" value="${special_connection if special_connection != '' else default_connection}" />
+      <xacro:ati_mini45_with_camera
+          parent_link="${arm_prefix_modified}${default_connection}"
+          prefix="${arm_prefix_modified}${arm_id}"
+          ip_address="$(arg ft_sensor_ip)"
+          gazebo="${gazebo}"
+          rpy_ee="$(arg rpy_ee)"
+          xyz_ee="$(arg xyz_ee)"
+          rdt_sampling_rate="$(arg rdt_sampling_rate)"
+          internal_filter_rate="$(arg internal_filter_rate)"
+          use_hardware_biasing="$(arg use_hardware_biasing)"
+          sensor_inertials="${xacro.load_yaml('$(find franka_description)/end_effectors/$(arg ee_id)/inertials.yaml')}"
+          measurement_frame_name="${ft_sensor_measurement_frame_name}" />
+    </xacro:if>
+    <xacro:if value="${hand and ee_id != 'none' and ee_id != 'franka_hand' and ee_id != 'ati_mini45_with_camera'}">
       <xacro:include filename="$(find franka_description)/end_effectors/common/ee_with_one_link.xacro"/>
       <xacro:include filename="$(find franka_description)/end_effectors/common/utils.xacro" />
       <xacro:include filename="$(find franka_description)/end_effectors/$(arg ee_id)/$(arg ee_id)_arguments.xacro" />
       <xacro:property name="default_connection" value="${(arm_id + '_link8') if not use_ft_sensor else 'ati_mini45_tool_mount'}" />
-      <xacro:property name="connection" value="${special_connection if special_connection != '' else default_connection}" />
       <xacro:ee_with_one_link
-        connected_to="${arm_prefix_modified}${connection}"
+        connected_to="${arm_prefix_modified}${default_connection}"
         arm_id="${arm_id}"
         arm_prefix="${arm_prefix_modified}"
@@ -114,11 +134,11 @@
     </xacro:if>
     <!-- D435 camera -->
-    <!-- TODO: pass location of calibrated-params -->
+    <!-- TODO: pass location of calibrated_params -->
     <xacro:property name="camera_pose_file"
-                    value="$(find franka_description)/robots/${arm_id}/calibrated-params.yaml" />
+                    value="$(find franka_description)/end_effectors/$(arg ee_id)/calibrated_params.yaml" />
     <xacro:property name="camera_pose" value="${xacro.load_yaml(camera_pose_file)}"/>
     <link name="${arm_id}_ref_camera_link"/>
     <joint name="${arm_id}_ref_camera_joint" type="fixed">
-      <parent link="${arm_id}_hand"/>
+      <parent link="${camera_pose['camera']['parent_frame']}"/>
       <child link="${arm_id}_ref_camera_link"/>
       <origin xyz="${camera_pose['camera']['x']}
@@ -132,36 +152,38 @@
     <!-- use_mesh="true" produces an error when visualizing with rviz2
     because the generated urdf contains mesh filename paths that do not start with file:// -->
-    <xacro:sensor_d435 parent="${arm_id}_ref_camera_link" name="camera" use_nominal_extrinsics="true" use_mesh="false">
+    <xacro:sensor_d435 parent="${arm_id}_ref_camera_link" name="camera" use_nominal_extrinsics="true" use_mesh="true">
       <origin xyz="0 0 0" rpy="0 0 0"/>
     </xacro:sensor_d435>
     <!-- camera support -->
-    <link name="${arm_id}_camera_support_link">
-      <inertial>
-        <mass value="0.010"/>
-        <origin xyz="0 0 0"/>
-        <inertia ixx="0.001" iyy="0.001" izz="0.001" ixy="0" iyz="0" ixz="0"/>
-      </inertial>
-      <visual>
-        <origin xyz="0.022 0 -0.012" rpy="3.141592653589793 0 -1.5707963267948966"/>
-        <geometry>
-          <mesh filename="package://franka_description/meshes/camera-support.stl" />
-        </geometry>
-        <material name="camera_support">
-          <color rgba="0 0.0 0.0 1.0"/>
-        </material>
-      </visual>
-      <collision>
-        <origin xyz="0.022 0 -0.012" rpy="3.141592653589793 0 -1.5707963267948966"/>
-        <geometry>
-          <mesh filename="package://franka_description/meshes/camera-support.stl" />
-        </geometry>
-      </collision>
-    </link>
-    <joint name="${arm_id}_camera_support_joint" type="fixed">
-      <parent link="${arm_id}_hand"/>
-      <child link="${arm_id}_camera_support_link"/>
-      <origin xyz="0 0 0" rpy="3.141592653589793 0 0"/>
-    </joint>
-    <!-- Definition of additional Gazebo tags -->
+     <xacro:unless value="${ee_id == 'ati_mini45_with_camera'}">
+       <link name="${arm_id}_camera_support_link">
+         <inertial>
+           <mass value="0.010"/>
+           <origin xyz="0 0 0"/>
+           <inertia ixx="0.001" iyy="0.001" izz="0.001" ixy="0" iyz="0" ixz="0"/>
+         </inertial>
+         <visual>
+           <origin xyz="0.022 0 -0.012" rpy="${pi} 0 -${pi / 2}"/>
+           <geometry>
+             <mesh filename="package://franka_description/meshes/camera_support.stl" />
+           </geometry>
+           <material name="camera_support">
+             <color rgba="0 0.0 0.0 1.0"/>
+           </material>
+         </visual>
+         <collision>
+           <origin xyz="0.022 0 -0.012" rpy="${pi} 0 -${pi / 2}"/>
+           <geometry>
+             <mesh filename="package://franka_description/meshes/camera_support.stl" />
+           </geometry>
+         </collision>
+       </link>
+       <joint name="${arm_id}_camera_support_joint" type="fixed">
+         <parent link="${camera_pose['camera']['parent_frame']}"/>
+         <child link="${arm_id}_camera_support_link"/>
+         <origin xyz="0 0 0" rpy="${pi} 0 0"/>
+       </joint>
+     </xacro:unless>
+     <!-- Definition of additional Gazebo tags -->
     <xacro:if value="${gazebo}">
       <xacro:if value="${parent != ''}">

Commit message: Add no camera ft sensor variant and option to disable camera

File: robots/common/franka_robot.xacro (robot description, xacro)
@@ -24,5 +24,6 @@
                       connected_to:='base'
                       multi_arm:=false
-                      use_ft_sensor:='false'">
+                      use_ft_sensor:='false'
+                      use_camera:='false'">
     <xacro:include filename="$(find franka_description)/robots/common/utils.xacro" />
     <xacro:include filename="$(find franka_description)/robots/common/franka_arm.xacro" />
@@ -45,5 +46,5 @@
     <xacro:if value="${use_ft_sensor}">
       <xacro:property name="ft_sensor_measurement_frame_name" value="${arm_prefix_modified}ati_mini45_measurement_reference" />
-      <xacro:if value="${hand and ee_id != 'ati_mini45_with_camera'}">
+      <xacro:if value="${hand and ee_id != 'ati_mini45_with_camera' and ee_id != 'ati_mini45_no_camera'}">
         <xacro:include filename="$(find franka_description)/end_effectors/ft_sensors/ati_mini45.urdf.xacro" />
         <xacro:include filename="$(find franka_description)/end_effectors/ft_sensors/ati_mini45_arguments.xacro" />
@@ -111,5 +112,24 @@
           with_sc="${with_sc}" />
     </xacro:if>
-    <xacro:if value="${hand and ee_id != 'none' and ee_id != 'franka_hand' and ee_id != 'ati_mini45_with_camera'}">
+    <xacro:if value="${hand and ee_id == 'ati_mini45_no_camera'}">
+      <xacro:include filename="$(find franka_description)/end_effectors/common/utils.xacro" />
+      <xacro:include filename="$(find franka_description)/end_effectors/$(arg ee_id)/$(arg ee_id).urdf.xacro" />
+      <xacro:include filename="$(find franka_description)/end_effectors/$(arg ee_id)/$(arg ee_id)_arguments.xacro" />
+      <xacro:property name="default_connection" value="${arm_id + '_link8'}" />
+      <xacro:ati_mini45_no_camera
+          parent_link="${arm_prefix_modified}${default_connection}"
+          prefix="${arm_prefix_modified}${arm_id}"
+          ip_address="$(arg ft_sensor_ip)"
+          gazebo="${gazebo}"
+          rpy_ee="$(arg rpy_ee)"
+          xyz_ee="$(arg xyz_ee)"
+          rdt_sampling_rate="$(arg rdt_sampling_rate)"
+          internal_filter_rate="$(arg internal_filter_rate)"
+          use_hardware_biasing="$(arg use_hardware_biasing)"
+          sensor_inertials="${xacro.load_yaml('$(find franka_description)/end_effectors/$(arg ee_id)/inertials.yaml')}"
+          measurement_frame_name="${ft_sensor_measurement_frame_name}"
+          with_sc="${with_sc}" />
+    </xacro:if>
+    <xacro:if value="${hand and ee_id != 'none' and ee_id != 'franka_hand' and ee_id != 'ati_mini45_with_camera' and ee_id != 'ati_mini45_no_camera'}">
       <xacro:include filename="$(find franka_description)/end_effectors/common/ee_with_one_link.xacro"/>
       <xacro:include filename="$(find franka_description)/end_effectors/common/utils.xacro" />
@@ -132,56 +152,58 @@
       />
     </xacro:if>
-    <!-- D435 camera -->
-    <!-- TODO: pass location of calibrated_params -->
-    <xacro:property name="camera_pose_file"
-                    value="$(find franka_description)/end_effectors/$(arg ee_id)/calibrated_params.yaml" />
-    <xacro:property name="camera_pose" value="${xacro.load_yaml(camera_pose_file)}"/>
-    <link name="${arm_id}_ref_camera_link"/>
-    <joint name="${arm_id}_ref_camera_joint" type="fixed">
-      <parent link="${camera_pose['camera']['parent_frame']}"/>
-      <child link="${arm_id}_ref_camera_link"/>
-      <origin xyz="${camera_pose['camera']['x']}
-                    ${camera_pose['camera']['y']}
-                    ${camera_pose['camera']['z']}"
-        rpy="${camera_pose['camera']['roll']}
-                    ${camera_pose['camera']['pitch']}
-                    ${camera_pose['camera']['yaw']}"/>
-    </joint>
-    <xacro:include filename="$(find realsense2_description)/urdf/_d435.urdf.xacro" />
-    <!-- use_mesh="true" produces an error when visualizing with rviz2
-    because the generated urdf contains mesh filename paths that do not start with file:// -->
-    <xacro:sensor_d435 parent="${arm_id}_ref_camera_link" name="camera" use_nominal_extrinsics="true" use_mesh="true">
-      <origin xyz="0 0 0" rpy="0 0 0"/>
-    </xacro:sensor_d435>
-    <!-- camera support -->
-     <xacro:unless value="${ee_id == 'ati_mini45_with_camera'}">
-       <link name="${arm_id}_camera_support_link">
-         <inertial>
-           <mass value="0.010"/>
-           <origin xyz="0 0 0"/>
-           <inertia ixx="0.001" iyy="0.001" izz="0.001" ixy="0" iyz="0" ixz="0"/>
-         </inertial>
-         <visual>
-           <origin xyz="0.022 0 -0.012" rpy="${pi} 0 -${pi / 2}"/>
-           <geometry>
-             <mesh filename="package://franka_description/meshes/camera_support.stl" />
-           </geometry>
-           <material name="camera_support">
-             <color rgba="0 0.0 0.0 1.0"/>
-           </material>
-         </visual>
-         <collision>
-           <origin xyz="0.022 0 -0.012" rpy="${pi} 0 -${pi / 2}"/>
-           <geometry>
-             <mesh filename="package://franka_description/meshes/camera_support.stl" />
-           </geometry>
-         </collision>
-       </link>
-       <joint name="${arm_id}_camera_support_joint" type="fixed">
-         <parent link="${camera_pose['camera']['parent_frame']}"/>
-         <child link="${arm_id}_camera_support_link"/>
-         <origin xyz="0 0 0" rpy="${pi} 0 0"/>
-       </joint>
-     </xacro:unless>
+    <xacro:if value="${use_camera}">
+      <!-- D435 camera -->
+      <!-- TODO: pass location of calibrated_params -->
+      <xacro:property name="camera_pose_file"
+                      value="$(find franka_description)/end_effectors/$(arg ee_id)/calibrated_params.yaml" />
+      <xacro:property name="camera_pose" value="${xacro.load_yaml(camera_pose_file)}"/>
+      <link name="${arm_id}_ref_camera_link"/>
+      <joint name="${arm_id}_ref_camera_joint" type="fixed">
+        <parent link="${camera_pose['camera']['parent_frame']}"/>
+        <child link="${arm_id}_ref_camera_link"/>
+        <origin xyz="${camera_pose['camera']['x']}
+                      ${camera_pose['camera']['y']}
+                      ${camera_pose['camera']['z']}"
+          rpy="${camera_pose['camera']['roll']}
+                      ${camera_pose['camera']['pitch']}
+                      ${camera_pose['camera']['yaw']}"/>
+      </joint>
+      <xacro:include filename="$(find realsense2_description)/urdf/_d435.urdf.xacro" />
+      <!-- use_mesh="true" produces an error when visualizing with rviz2
+      because the generated urdf contains mesh filename paths that do not start with file:// -->
+      <xacro:sensor_d435 parent="${arm_id}_ref_camera_link" name="camera" use_nominal_extrinsics="true" use_mesh="true">
+        <origin xyz="0 0 0" rpy="0 0 0"/>
+      </xacro:sensor_d435>
+      <!-- camera support -->
+      <xacro:unless value="${ee_id == 'ati_mini45_with_camera'}">
+        <link name="${arm_id}_camera_support_link">
+          <inertial>
+            <mass value="0.010"/>
+            <origin xyz="0 0 0"/>
+            <inertia ixx="0.001" iyy="0.001" izz="0.001" ixy="0" iyz="0" ixz="0"/>
+          </inertial>
+          <visual>
+            <origin xyz="0.022 0 -0.012" rpy="${pi} 0 -${pi / 2}"/>
+            <geometry>
+              <mesh filename="package://franka_description/meshes/camera_support.stl" />
+            </geometry>
+            <material name="camera_support">
+              <color rgba="0 0.0 0.0 1.0"/>
+            </material>
+          </visual>
+          <collision>
+            <origin xyz="0.022 0 -0.012" rpy="${pi} 0 -${pi / 2}"/>
+            <geometry>
+              <mesh filename="package://franka_description/meshes/camera_support.stl" />
+            </geometry>
+          </collision>
+        </link>
+        <joint name="${arm_id}_camera_support_joint" type="fixed">
+          <parent link="${camera_pose['camera']['parent_frame']}"/>
+          <child link="${arm_id}_camera_support_link"/>
+          <origin xyz="0 0 0" rpy="${pi} 0 0"/>
+        </joint>
+      </xacro:unless>
+     </xacro:if>
      <!-- Definition of additional Gazebo tags -->
     <xacro:if value="${gazebo}">

File: robots/fer/fer.urdf.xacro (robot description, xacro)
@@ -41,4 +41,6 @@
   <!-- Should force torque sensors be used? -->
   <xacro:arg name="use_ft_sensor" default="false" />
+  <!-- Should RealSense d435i be loaded? -->
+  <xacro:arg name="use_camera" default="false" />
   <xacro:franka_robot arm_id="fer"
                       joint_limits="${xacro.load_yaml('$(find franka_description)/robots/fer/joint_limits.yaml')}"
@@ -59,5 +61,6 @@
                       arm_prefix=""
                       connected_to="base"
-                      use_ft_sensor="$(arg use_ft_sensor)">
+                      use_ft_sensor="$(arg use_ft_sensor)"
+                      use_camera="$(arg use_camera)">
   </xacro:franka_robot>
 </robot>
