Commit message: Add initial setup for the mini camera mount

File: robots/common/franka_robot.xacro (robot description, xacro)
@@ -48,5 +48,5 @@
     <xacro:if value="${use_ft_sensor}">
       <xacro:property name="ft_sensor_measurement_frame_name" value="${arm_prefix_modified}ati_mini45_measurement_reference" />
-      <xacro:if value="${hand and ee_id != 'ati_mini45_with_camera' and ee_id != 'ati_mini45_no_camera'}">
+      <xacro:if value="${hand and 'ati_mini45' not in ee_id}">
         <xacro:include filename="$(find franka_description)/end_effectors/ft_sensors/ati_mini45.urdf.xacro" />
         <xacro:include filename="$(find franka_description)/end_effectors/ft_sensors/ati_mini45_arguments.xacro" />
@@ -133,5 +133,24 @@
           with_sc="${with_sc}" />
     </xacro:if>
-    <xacro:if value="${hand and ee_id != 'none' and ee_id != 'franka_hand' and ee_id != 'ati_mini45_with_camera' and ee_id != 'ati_mini45_no_camera'}">
+    <xacro:if value="${hand and ee_id == 'ati_mini45_with_compact_camera'}">
+      <xacro:include filename="$(find franka_description)/end_effectors/common/utils.xacro" />
+      <xacro:include filename="$(find franka_description)/end_effectors/$(arg ee_id)/$(arg ee_id).urdf.xacro" />
+      <xacro:include filename="$(find franka_description)/end_effectors/$(arg ee_id)/$(arg ee_id)_arguments.xacro" />
+      <xacro:property name="default_connection" value="${arm_id + '_link8'}" />
+      <xacro:ati_mini45_with_compact_camera
+          parent_link="${arm_prefix_modified}${default_connection}"
+          prefix="${arm_prefix_modified}${arm_id}"
+          ip_address="$(arg ft_sensor_ip)"
+          gazebo="${gazebo}"
+          rpy_ee="$(arg rpy_ee)"
+          xyz_ee="$(arg xyz_ee)"
+          rdt_sampling_rate="$(arg rdt_sampling_rate)"
+          internal_filter_rate="$(arg internal_filter_rate)"
+          use_hardware_biasing="$(arg use_hardware_biasing)"
+          sensor_inertials="${xacro.load_yaml('$(find franka_description)/end_effectors/$(arg ee_id)/inertials.yaml')}"
+          measurement_frame_name="${ft_sensor_measurement_frame_name}"
+          with_sc="${with_sc}" />
+    </xacro:if>
+    <xacro:if value="${hand and ee_id != 'none' and ee_id != 'franka_hand' and 'ati_mini45' not in ee_id}">
       <xacro:include filename="$(find franka_description)/end_effectors/common/ee_with_one_link.xacro"/>
       <xacro:include filename="$(find franka_description)/end_effectors/common/utils.xacro" />
@@ -178,5 +197,5 @@
       </xacro:sensor_d435>
       <!-- camera support -->
-      <xacro:unless value="${ee_id == 'ati_mini45_with_camera'}">
+      <xacro:unless value="${ee_id == 'ati_mini45_with_camera' or ee_id == 'ati_mini45_with_compact_camera'}">
         <link name="${arm_id}_camera_support_link">
           <inertial>
