Commit message: Tune capsules | Move camera capsule to the robot section

File: end_effectors/ati_mini45_with_compact_camera/ati_mini45_with_compact_camera.urdf.xacro (robot description, xacro)
@@ -30,7 +30,4 @@
       </collision>
       <xacro:ee-inertials name="ati_mini45_with_compact_camera_base" />
-      <xacro:if value="${with_sc}">
-        <xacro:collision_capsule xyz="0.12 0 -0.05" direction="y" radius="${0.04+safety_distance}" length="0.08" />
-      </xacro:if>
     </link>
     <!-- sub-link defining coarse geometries of real end-effector's internal self-collision -->
@@ -38,5 +35,5 @@
       <link name="${prefix_expanded}ati_mini45_with_compact_camera_sc">
         <xacro:unless value="${gazebo}">
-          <xacro:collision_capsule xyz="0 0 ${length / 2}" direction="y" radius="${radius+safety_distance}" length="${length}" />
+          <xacro:collision_capsule xyz="0 0 ${length / 2}" direction="z" radius="${radius+safety_distance}" length="${length}" />
         </xacro:unless>
       </link>
@@ -67,5 +64,5 @@
       <xacro:ee-inertials name="ati_mini45_with_compact_camera_tool" />
       <xacro:if value="${with_sc}">
-        <xacro:collision_capsule xyz="0 0 -0.01" direction="z" radius="${0.015+safety_distance}" length="0.02" />
+        <xacro:collision_capsule xyz="0 0 -0.02" direction="z" radius="${0.012+safety_distance}" length="0.1" />
       </xacro:if>
     </link>

File: robots/common/franka_arm.xacro (robot description, xacro)
@@ -109,6 +109,6 @@
     <xacro:link_with_sc no_prefix="${no_prefix}" name="link7" gazebo="${gazebo}" rpy="0 0 ${pi/4}" with_sc="${with_sc}">
       <self_collision_geometries>
-        <xacro:collision_capsule xyz="0 0 0.035" direction="z" radius="${0.045+safety_distance}" length="0.31" />
-        <xacro:collision_capsule xyz="0.05 0 0.082" direction="x" radius="${0.03+safety_distance}" length="0.05" />
+        <xacro:collision_capsule xyz="0 0 0.02" direction="z" radius="${0.045+safety_distance}" length="0.28" />
+        <xacro:collision_capsule xyz="0.06 0 0.082" direction="y" radius="${0.03+safety_distance}" length="0.05" />
       </self_collision_geometries>
     </xacro:link_with_sc>

File: robots/common/franka_robot.xacro (robot description, xacro)
@@ -179,5 +179,9 @@
                       value="$(find franka_description)/end_effectors/$(arg ee_id)/${arm_id}/calibrated_params.yaml" />
       <xacro:property name="camera_pose" value="${xacro.load_yaml(camera_pose_file)}"/>
-      <link name="${arm_id}_ref_camera_link"/>
+      <link name="${arm_id}_ref_camera_link">
+        <xacro:if value="${with_sc}">
+          <xacro:collision_capsule xyz="0.002 0 0.012" direction="y" radius="${0.015+robot_safety_distance}" length="0.13" />
+        </xacro:if>
+      </link>
       <joint name="${arm_id}_ref_camera_joint" type="fixed">
         <parent link="${camera_pose['camera']['parent_frame']}"/>

Commit message: Update origin of the tip

File: end_effectors/ati_mini45_with_compact_camera/ati_mini45_with_compact_camera.urdf.xacro (robot description, xacro)
@@ -54,5 +54,5 @@
       <parent link="${measurement_frame_name}" />
       <child link="${prefix_expanded}ati_mini45_with_compact_camera_tool" />
-      <origin xyz="0 0 -0.073915" rpy="${pi} 0.0 ${pi / 3 * 2}" />
+      <origin xyz="0 0 -0.07885" rpy="${pi} 0.0 ${pi / 3 * 2}" />
     </joint>
     <link name="${prefix_expanded}ati_mini45_with_compact_camera_tool">
